Commit message: Fix URDF: material naming, hip axis convention, limit tuning, add README

File: urdf/dog_urdf.urdf (robot description, URDF)
Before this commit: robot dog_urdf, 17 links, 16 joints
Joints:
- joint FL_foot_joint: axis 0 0 0 -> (none)
- joint FL_hip_joint: limit lower=-0.65 upper=0.65 effort=40 velocity=12 -> lower=-0.5 upper=0.5 effort=40 velocity=12
- joint FR_foot_joint: axis 0 0 0 -> (none)
- joint FR_hip_joint: axis 1 0 0 -> -1 0 0; limit lower=-0.65 upper=0.65 effort=40 velocity=12 -> lower=-0.5 upper=0.5 effort=40 velocity=12
- joint RL_foot_joint: axis 0 0 0 -> (none)
- joint RL_hip_joint: axis -1 0 0 -> 1 0 0; limit lower=-0.65 upper=0.65 effort=40 velocity=12 -> lower=-0.5 upper=0.5 effort=40 velocity=12
- joint RR_foot_joint: axis 0 0 0 -> (none)
- joint RR_hip_joint: limit lower=-0.65 upper=0.65 effort=40 velocity=12 -> lower=-0.5 upper=0.5 effort=40 velocity=12

Commit message: fix: ROS2 migration, capsule→cylinder, add Gazebo ros2_control tags

File: urdf/dog_urdf.urdf (robot description, URDF)
Before this commit: robot dog_urdf, 17 links, 16 joints
Links:
- link FL_calf: geometry collision cylinder length=0.18 radius=0.022; visual mesh filename=package://dog_urdf/meshes/FL_calf.STL
- link FL_thigh: geometry collision cylinder length=0.18 radius=0.03; visual mesh filename=package://dog_urdf/meshes/FL_thigh.STL
- link FR_calf: geometry collision cylinder length=0.18 radius=0.022; visual mesh filename=package://dog_urdf/meshes/FR_calf.STL
- link FR_thigh: geometry collision cylinder length=0.18 radius=0.03; visual mesh filename=package://dog_urdf/meshes/FR_thigh.STL
- link RL_calf: geometry collision cylinder length=0.18 radius=0.022; visual mesh filename=package://dog_urdf/meshes/RL_calf.STL
- link RL_thigh: geometry collision cylinder length=0.18 radius=0.03; visual mesh filename=package://dog_urdf/meshes/RL_thigh.STL
- link RR_calf: geometry collision cylinder length=0.18 radius=0.022; visual mesh filename=package://dog_urdf/meshes/RR_calf.STL
- link RR_thigh: geometry collision cylinder length=0.18 radius=0.03; visual mesh filename=package://dog_urdf/meshes/RR_thigh.STL

Commit message: fix: widen joint limits to match actual hardware operating range
Previous limits were narrower than the hardware's q_min/q_max range,
causing gait_position_controller to clamp during lie-down (motor→0
maps to thigh=1.254 rad, calf=-2.791 rad in URDF frame).

thigh: [-1.6, 0.8] → [-1.90, 1.92]
calf:  [-2.4, -0.3] → [-2.80, -0.28]

Derived from robot.yaml: q_urdf = direction * q_motor + zero_offset

File: urdf/dog_urdf.urdf (robot description, URDF)
Before this commit: robot dog_urdf, 17 links, 16 joints
Joints:
- joint FL_calf_joint: limit lower=-2.4 upper=-0.3 effort=55 velocity=14 -> lower=-2.80 upper=-0.28 effort=55 velocity=14
- joint FL_thigh_joint: limit lower=-1.6 upper=0.8 effort=55 velocity=14 -> lower=-1.90 upper=1.92 effort=55 velocity=14
- joint FR_calf_joint: limit lower=-2.4 upper=-0.3 effort=55 velocity=14 -> lower=-2.80 upper=-0.28 effort=55 velocity=14
- joint FR_thigh_joint: limit lower=-1.6 upper=0.8 effort=55 velocity=14 -> lower=-1.90 upper=1.92 effort=55 velocity=14
- joint RL_calf_joint: limit lower=-2.4 upper=-0.3 effort=55 velocity=14 -> lower=-2.80 upper=-0.28 effort=55 velocity=14
- joint RL_thigh_joint: limit lower=-1.6 upper=0.8 effort=55 velocity=14 -> lower=-1.90 upper=1.92 effort=55 velocity=14
- joint RR_calf_joint: limit lower=-2.4 upper=-0.3 effort=55 velocity=14 -> lower=-2.80 upper=-0.28 effort=55 velocity=14
- joint RR_thigh_joint: limit lower=-1.6 upper=0.8 effort=55 velocity=14 -> lower=-1.90 upper=1.92 effort=55 velocity=14

Commit message: feat(urdf): add depth camera sensor for Gazebo simulation

File: urdf/dog_urdf.urdf (robot description, URDF)
Before this commit: robot dog_urdf, 17 links, 16 joints
Links:
- added link camera_depth_optical_frame
Joints:
- added joint camera_depth_joint: type fixed, parent base_link, child camera_depth_optical_frame, origin xyz=0.15 0 0.12 rpy=-1.5707963 0 -1.5707963

Commit message: feat(urdf): add camera_link and odin1_base_link fixed joints

File: urdf/dog_urdf.urdf (robot description, URDF)
Before this commit: robot dog_urdf, 18 links, 17 joints
Links:
- added link camera_link
- added link odin1_base_link
Joints:
- added joint camera_joint: type fixed, parent base_link, child camera_link, origin xyz=0.15 0 0.12 rpy=0 0.5236 0
- added joint odin1_base_joint: type fixed, parent base_link, child odin1_base_link, origin xyz=0.10 0 0.08 rpy=0 0 0

Commit message: fix(urdf): remove odin1_base_link fixed joint to avoid TF conflict

File: urdf/dog_urdf.urdf (robot description, URDF)
Before this commit: robot dog_urdf, 20 links, 19 joints
Links:
- removed link odin1_base_link
Joints:
- removed joint odin1_base_joint

Commit message: fix(urdf): update camera mount to measured position (x=0.238 y=-0.012 z=0.068)

File: urdf/dog_urdf.urdf (robot description, URDF)
Before this commit: robot dog_urdf, 19 links, 18 joints
Joints:
- joint camera_joint: origin xyz=0.15 0 0.12 rpy=0 0.5236 0 -> xyz=0.238 -0.012 0.068 rpy=0 0.5236 0
